Commit message: Format and add contact tags to robotiq urdf

File: corallab_sim/robots/assets/ur5/gripper/robotiq_2f_85.urdf (robot description, URDF)
Before this commit: robot example, 12 links, 11 joints
Links:
- added link robotiq_2f_85_grasp_target, mass 0.0
Joints:
- added joint robotiq_2f_85_grasp_target_joint: type fixed, parent robotiq_2f_85_base, child robotiq_2f_85_grasp_target, origin xyz=0 0 0.105 rpy=0 0 0

Commit message: Better grasping by detecting contact force. Add draw_text util.

File: corallab_sim/robots/assets/ur5/gripper/robotiq_2f_85.urdf (robot description, URDF)
Before this commit: robot example, 13 links, 12 joints
Joints:
- joint robotiq_2f_85_right_driver_joint: limit lower=0.0 upper=0.834 effort=60 velocity=1.91986177778 -> lower=0.0 upper=0.834 effort=20 velocity=1.91986177778
